File: ESP32_IoT_Board.kicad_sch (KiCad schematic)
At the start: 25 parts, among them J1 SS-52400-002, J2 B2B-PH-SM4-TB, U1 MCP73871-2CAI_ML

Commit message: SCH completed
Other:
- sheet ESP32-C3-02 ports: added USB_DN, USB_DP, VBAT; removed none
Changed lines of the file:
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@@
 	(wire
 		(pts
+			(xy 165.1 127) (xy 168.91 127)
+		)
+		(stroke
+			(width 0)
+			(type default)
+		)
+	)
+	(wire
+		(pts
 			(xy 101.6 170.18) (xy 111.76 170.18)
 		)
@@
 	(wire
 		(pts
+			(xy 165.1 130.81) (xy 168.91 130.81)
+		)
+		(stroke
+			(width 0)
+			(type default)
+		)
+	)
+	(wire
+		(pts
 			(xy 212.725 34.29) (xy 212.725 36.83)
 		)
@@
 	(wire
 		(pts
+			(xy 165.1 123.19) (xy 168.91 123.19)
+		)
+		(stroke
+			(width 0)
+			(type default)
+		)
+	)
+	(wire
+		(pts
 			(xy 182.88 44.45) (xy 182.88 52.07)
 		)
@@
 	)
 	(label "USB_DP"
+		(at 168.91 127 0)
+		(effects
+			(font
+				(size 1.27 1.27)
+			)
+			(justify left bottom)
+		)
+	)
+	(label "USB_DP"
 		(at 39.37 43.18 180)
 		(effects
@@
 	)
 	(label "USB_DN"
+		(at 168.91 123.19 0)
+		(effects
+			(font
+				(size 1.27 1.27)
+			)
+			(justify left bottom)
+		)
+	)
+	(label "VBUS"
+		(at 168.91 130.81 0)
+		(effects
+			(font
+				(size 1.27 1.27)
+			)
+			(justify left bottom)
+		)
+	)
+	(label "USB_DN"
 		(at 80.01 45.72 0)
 		(effects
@@
 			)
 		)
+		(pin "USB_DN" input
+			(at 165.1 123.19 0)
+			(effects
+				(font
+					(size 1.27 1.27)
+				)
+				(justify right)
+			)
+		)
+		(pin "USB_DP" input
+			(at 165.1 127 0)
+			(effects
+				(font
+					(size 1.27 1.27)
+				)
+				(justify right)
+			)
+		)
+		(pin "VBAT" input
+			(at 165.1 130.81 0)
+			(effects
+				(font
+					(size 1.27 1.27)
+				)
+				(justify right)
+			)
+		)

Commit message: clean Warnings on the SCH
Parts:
- C1, C2, C5, C6: footprint (none) -> Capacitor_SMD:C_0805_2012Metric_Pad1.18x1.45mm_HandSolder
- C3, C4: footprint (none) -> Capacitor_Tantalum_SMD:CP_EIA-3216-10_Kemet-I_HandSolder
- F1: footprint FUSC3226X100N -> ESP32 Project Libraries:FUSC3226X100N
- J1: footprint SS-52400-002:BELFUSE_SS-52400-002 -> ESP32 Project Libraries:BELFUSE_SS-52400-002
- J2: footprint B2B-PH-SM4-TB:JST_B2B-PH-SM4-TB -> ESP32 Project Libraries:JST_B2B-PH-SM4-TB
- LED1, LED2, LED3, LED4: footprint LEDC2012X120N -> ESP32 Project Libraries:LEDC2012X120N
- R1, R10, R2, R3, R4, R5, R6, R7, R8, R9: footprint (none) -> Resistor_SMD:R_0805_2012Metric_Pad1.20x1.40mm_HandSolder
- U1: footprint MCP73871-2CAI_ML:QFN50P400X400X100-21N -> ESP32 Project Libraries:QFN50P400X400X100-21N
- U8: renamed from VR1; footprint LM1117MPX-3.3:VREG_LM1117MPX-3.3 -> ESP32 Project Libraries:VREG_LM1117MPX-3.3
Connections:
- net GND: now also U1.3 (SEL)

Commit message: PCB completed
Parts:
- added F2: 0ZCH0110AF2E, ESP32 Project Libraries:FUSC3226X100N, symbol 0ZCH0110AF2E:0ZCH0110AF2E
Connections:
- net +5V: now also F2.2; no longer U1.1 (OUT), U1.20 (OUT)
- new net: F2.1, U1.1 (OUT), U1.20 (OUT)
Other:
- moved on the sheet: C6, LED1, LED2, LED3, R1, R2, R5, R6, R7, R8, R9, U1
