File: ESP32_IoT_Board.kicad_pcb (KiCad board)
At the start: 4 copper layers, 87 parts, among them J1 SS-52400-002, J2 B2B-PH-SM4-TB, J3 GSD090012SEU, J4 Conn_01x04_Pin, J5 Conn_01x05_Pin, Q1 TEMT6000X01, Q2 BC817, Q3 BC817, U1 MCP73871-2CAI_ML, U2 BME280, U3 ESP32-C3-WROOM-02-H4, U4 CP2102N-Axx-xQFN20, U5 USBLC6-2SC6, U6 W25Q32JVSSIQ, U7 MAX4466EXK, U8 LM1117MPX-3.3

Commit message: PCB completed
Parts:
- removed J5: Conn_01x05_Pin, Connector_PinHeader_2.54mm:PinHeader_1x05_P2.54mm_Vertical
- added C23: 0.1u, Capacitor_SMD:C_0805_2012Metric_Pad1.18x1.45mm_HandSolder, F.Cu at (95.7, 36.4)
- added C24: 10n, Capacitor_SMD:C_0805_2012Metric_Pad1.18x1.45mm_HandSolder, F.Cu at (91.2, 32.8)
- added C25: 10n, Capacitor_SMD:C_0805_2012Metric_Pad1.18x1.45mm_HandSolder, F.Cu at (152.4, 36.7)
- added F2: 0ZCH0110AF2E, ESP32 Project Libraries:FUSC3226X100N, F.Cu at (52.9, 86.3)
- added G***: LOGO, Logo:TP_Logo_New_10mm_Positive, F.Cu at (92.5, 64.0)
- added LED7: LTST-C170KRKT, ESP32 Project Libraries:LEDC2012X120N, F.Cu at (94.3, 83.3)
- added LED8: LTST-C170GKT, ESP32 Project Libraries:LEDC2012X120N, F.Cu at (88.8, 83.3)
- added R17: 35WR100KLFTR, ESP32 Project Libraries:TRIM_35WR100KLFTR, F.Cu at (61.1, 40.6)
- added R36: 10k, Resistor_SMD:R_0805_2012Metric_Pad1.20x1.40mm_HandSolder, F.Cu at (89.0, 75.8)
- added R37: 470, Resistor_SMD:R_0805_2012Metric_Pad1.20x1.40mm_HandSolder, F.Cu at (89.0, 79.3)
- added R38: 470, Resistor_SMD:R_0805_2012Metric_Pad1.20x1.40mm_HandSolder, F.Cu at (94.3, 79.3)
- added S3: SW1, ESP32 Project Libraries:SW_TL3305AF260QG, F.Cu at (83.2, 79.8)
- C28: value 1u -> 10u
- R30: value 10k -> 1k
- R31: value 100k -> 22k
- S1, S2: footprint ESP32 Project Libraries:SW_USLPT2819DT2TR -> ESP32 Project Libraries:SW_TL3305AF260QG
- moved F1 212.9 mm to (61.4, 71.0), turned to 90 degrees
- moved C1 206.7 mm to (72.1, 71.0), turned to -90 degrees
- moved J1 203.6 mm to (71.5, 84.9)
- moved R4 200.8 mm to (63.7, 80.0), turned to 90 degrees
- moved R3 198.3 mm to (63.5, 86.3), turned to 90 degrees
- moved U5 192.2 mm to (67.0, 70.8), turned to -90 degrees
- moved LED5 181.2 mm to (60.5, 57.8), turned to 90 degrees
- moved R14 180.3 mm to (60.6, 63.6), turned to -90 degrees
- moved R18 178.8 mm to (64.2, 63.6), turned to -90 degrees
- moved U4 178.6 mm to (70.2, 63.7), turned to 90 degrees
- moved LED6 178.3 mm to (64.3, 57.9), turned to 90 degrees
- moved J2 174.8 mm to (39.5, 82.8)
- moved R11 170.3 mm to (70.0, 58.5)
- moved C9 168.8 mm to (78.0, 63.5), turned to 90 degrees
- moved TP7 168.0 mm to (105.2, 61.8)
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Connections:
- Q1 pad 1: GND -> /ESP32-C3-02/PHOTO_C
- Q1 pad 3: /ESP32-C3-02/PHOTO_C -> +3.3V
- Q3 pad 2: /ESP32-C3-02/BOOT -> /ESP32-C3-02/DTR
- Q3 pad 3: /ESP32-C3-02/DTR -> /ESP32-C3-02/BOOT
- R23 pad 1: +3.3V -> /ESP32-C3-02/PHOTO_C
- R23 pad 2: /ESP32-C3-02/PHOTO_C -> GND
- R31 pad 2: /ESP32-C3-02/MIC_OUT -> Net-(R17-Pad3)
- S1 pad 2: GND -> /ESP32-C3-02/BOOT
- S1 pad 3: /ESP32-C3-02/BOOT -> GND
- S2 pad 2: GND -> /ESP32-C3-02/EN
- S2 pad 3: /ESP32-C3-02/EN -> GND
- U1 pad 1: /+5V -> Net-(F2-Pad1)
- U1 pad 20: /+5V -> Net-(F2-Pad1)
- U3 pad 18: /ESP32-C3-02/CS_SD -> /ESP32-C3-02/MIC_OUT
- U3 pad 4: /ESP32-C3-02/MIC_OUT -> /ESP32-C3-02/CS_SD
Other:
- board outline added: 127.9 x 63.9 mm
- board text added: "CHARGED"
- board text added: "CHARGING"
- board text added: "CHARGING PWR OK"
- board text added: "ESP32-C3-02"
- board text added: "Environment"
- board text added: "Flash Memory"
- board text added: "GPIO"
- board text added: "GPIO 08"
- board text added: "GPIO 18"
- board text added: "GPIO 19"
- board text added: "LCD Display"
- board text added: "LiPO Charger"
- board text added: "Light Sensor"
- board text added: "PROTOTYPES"
- board text added: "RESET BOOT"
- board text added: "SD Card"
- board text added: "Sensor"
- board text added: "Sound Sensor"
- board text added: "TINKER"
- board text added: "USB"

Commit message: route completed
Parts:
- added H1: MountingHole, MountingHole:MountingHole_2.5mm, F.Cu at (24.8, 30.9)
- added H2: MountingHole, MountingHole:MountingHole_2.5mm, F.Cu at (24.8, 87.3)
- added H3: MountingHole, MountingHole:MountingHole_2.5mm, F.Cu at (157.6, 37.6)
- added H4: MountingHole, MountingHole:MountingHole_2.5mm, F.Cu at (157.6, 87.3)
- moved LED1 8.79 mm to (40.0, 67.8)
- moved R9 8.79 mm to (40.0, 73.8)
- moved C13 6.96 mm to (136.4, 56.4)
- moved LED3 4.36 mm to (35.8, 67.9)
- moved R7 4.36 mm to (35.8, 73.9)
- moved LED2 4.36 mm to (31.3, 67.9)
- moved R8 4.36 mm to (31.3, 73.9)
- moved TP4 3.60 mm to (148.8, 56.0)
- moved C12 2.34 mm to (136.5, 60.5)
- moved R19 2.34 mm to (142.3, 60.5)
- moved J3 1.35 mm to (137.6, 76.8)
- moved J1 1.04 mm to (71.6, 86.0)
- moved G*** 0.80 mm to (91.8, 64.0)
- moved C1 0.44 mm to (71.7, 71.0), turned to 90 degrees
- moved C21 0.30 mm to (114.8, 80.5), turned to 180 degrees
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Routing:
- net /ESP32-C3-02/SCL: track 0.00 -> 180.6 mm, vias 0 -> 6
- net /ESP32-C3-02/SDA: track 0.00 -> 165.0 mm, vias 0 -> 2
- net /ESP32-C3-02/EN: track 0.00 -> 138.0 mm
- net /ESP32-C3-02/MIC_OUT: track 0.00 -> 124.2 mm, vias 0 -> 2
- net /ESP32-C3-02/GPIO18: track 0.00 -> 120.4 mm, vias 0 -> 2
- net /ESP32-C3-02/GPIO19: track 0.00 -> 114.1 mm, vias 0 -> 2
- net /ESP32-C3-02/RX_TX: track 0.00 -> 96.8 mm, vias 0 -> 2
- net /ESP32-C3-02/TX_RX: track 0.00 -> 94.3 mm, vias 0 -> 4
- net GND: track 0.00 -> 89.4 mm, vias 0 -> 57
- net /ESP32-C3-02/GPIO08: track 0.00 -> 77.0 mm, vias 0 -> 2
- net /+5V: track 0.00 -> 74.0 mm, vias 0 -> 2
- net /ESP32-C3-02/PHOTO_C: track 0.00 -> 69.7 mm, vias 0 -> 2
- net /ESP32-C3-02/BOOT: track 0.00 -> 68.6 mm, vias 0 -> 2
- net /ESP32-C3-02/RTS: track 0.00 -> 67.2 mm, vias 0 -> 2
- net /+5V_USB: track 0.00 -> 60.6 mm, vias 0 -> 5
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- added copper zone on F.Cu, net +3.3V
- added copper zone on In1.Cu, net +3.3V
- added copper zone on F.Cu, net /+5V
- added copper zone on F.Cu, net /+5V_USB
- added copper zone on In1.Cu, net /+5V_USB
- added copper zone on F.Cu, net /VBAT
- added copper zone on F.Cu, net /VBUS
- added copper zone on In1.Cu, net /VBUS
- added copper zone on F.Cu, net GND
- added copper zone on In2.Cu, net GND
Other:
- board size 127.9 x 63.9 mm -> 139.5 x 63.2 mm
