File: esp32-c3-02.kicad_sch (KiCad schematic)
At the start: 5 parts, among them J3 GSD090012SEU, U3 ESP32-C3-WROOM-02-H4, U4 CP2102N-Axx-xQFN20, U5 USBLC6-2SC6, U6 W25Q32JVSSIQ

Commit message: SCH completed
Parts:
- added C10, C13, C14, C8: 0.1u, symbol Device:C
- added C11: 1u, symbol Device:C
- added C12, C7: 10u, symbol Device:C_Polarized
- added C9: 4.7u, symbol Device:C_Polarized
- added LED5: LTST-C170GKT, LEDC2012X120N, symbol LTST-C170GKT:LTST-C170GKT
- added LED6: LTST-C170KRKT, LEDC2012X120N, symbol LTST-C170KRKT:LTST-C170KRKT
- added R11: 1k, symbol Device:R
- added R12: 22k1, symbol Device:R
- added R13: 47k5, symbol Device:R
- added R14, R18: 470, symbol Device:R
- added R16, R20, R21, R22: 50, symbol Device:R
- added R19: 10k, symbol Device:R
- added TP1: Test MOSI, symbol Connector:TestPoint
- added TP2: Test MISO, symbol Connector:TestPoint
- added TP3: Test SCLK, symbol Connector:TestPoint
- added TP4: Test CS_SD, symbol Connector:TestPoint
- added TP5: Test CS, symbol Connector:TestPoint
- added TP6: Test SDA, symbol Connector:TestPoint
- added TP7: Test SCL, symbol Connector:TestPoint
Connections:
- net GND: now reaches U4.12 (GND), U4.21 (GND), U4.3 (GND)
- net GND: now also J3.3 (VSS1), J3.6 (VSS2), J3.8 (DAT1), J3.9 (DAT2), J3.G1 (SHIELD_GND), J3.G2 (SHIELD_GND), J3.G3 (SHIELD_GND), J3.G4 (SHIELD_GND), U3.19 (GND), U3.20 (GND), U3.21 (GND), U3.22 (GND), U3.23 (GND), U3.24 (GND), U3.25 (GND), U3.26 (GND), U3.27 (GND), U3.28 (GND), U3.29 (GND), U3.30 (GND), U3.31 (GND), U3.32 (GND), U3.33 (GND), U3.34 (GND), U3.35 (GND), U3.36 (GND), U3.37 (GND), U3.38 (GND), U3.39 (GND), U3.9 (GND), U5.2 (GND), U6.4 (GND), C10.1, C11.2, C12.2, C13.1, C14.1, C7.2, C8.1, C9.2, R13.1
- net DTR: now reaches U4.15 (~{CTS})
- net RTS: now reaches U4.16 (~{RTS})
- net RX_TX: now reaches U4.17 (RXD)
- net RX_TX: now also U3.12 (TXD)
- net TX_RX: now reaches U4.18 (TXD)
- net TX_RX: now also U3.11 (RXD)
- net at U4.19 (~{RXT}/GPIO.3): now also R18.2
- net at U4.20 (~{TXT}/GPIO.2): now also R14.2
- net USB_D+: now reaches U4.4 (D+)
- net USB_D+: now also U5.3 (I/O2)
- net USB_D-: now reaches U4.5 (D-)
- net USB_D-: now also U5.1 (I/O1)
- net +3.3V: now reaches U4.6 (VDD)
- net +3.3V: now also J3.4 (VDD1), U3.1 (3V3), U4.7 (VREGIN), U6.3 (~{WP}(IO2)), U6.7 (~{HOLD}/~{RESET}(IO3)), U6.8 (VCC), C10.2, C12.1, C13.2, C14.2, C7.1, C8.2, C9.1, LED5.2 (A), LED6.2 (A), R11.1, R19.1
- net at U4.8 (VBUS): now also C11.1, R12.1, R13.2
- net at U4.9 (~{RST}): now also R11.2
- net CS_SD: now reaches J3.1 (CD/DAT3)
- net CS_SD: now also U3.18 (IO0), R19.2, TP4.1
- net MOSI_DI: now reaches J3.2 (CMD)
- net MOSI_DI: now also U6.5 (DI(IO0)), R21.1, TP1.1
- net SCLK: now reaches J3.5 (CLK)
- net SCLK: now also U6.6 (CLK), R20.2, TP3.1
- net at J3.7 (DAT0): now also R16.1
- net CS: now reaches U3.10 (IO10)
- net CS: now also U6.1 (~{CS}), TP5.1
- net GPIO18: now reaches U3.13 (IO18)
- net GPIO19: now reaches U3.14 (IO19)
- net SCL: now reaches U3.15 (IO3)
- net SCL: now also TP7.1
- net MISO_DO: now reaches U3.16 (IO2)
- net MISO_DO: now also R16.2, R22.1, TP2.1
- net PHOTO_C: now reaches U3.17 (IO1)
- net EN: now reaches U3.2 (EN)
- net SDA: now reaches U3.3 (IO4)
- net SDA: now also TP6.1
- net MIC_OUT: now reaches U3.4 (IO5)
- net at U3.5 (IO6): now also R20.1
- net at U3.6 (IO7): now also R21.2
- net GPIO08: now reaches U3.7 (IO8)
- net BOOT: now reaches U3.8 (IO9)
- net at U6.2 (DO(IO1)): now also R22.2
- net USB_DP: now reaches U5.4 (I/O2)
- net VBAT: now reaches U5.5 (VBUS)
- net VBAT: now also R12.2
- net USB_DN: now reaches U5.6 (I/O1)
- new net: LED6.1 (K), R18.1
- new net: LED5.1 (K), R14.1
- no-connect marks 0 -> 7
Other:
- added sheet Sensors (sensors.kicad_sch)
- added sheet User Interface (user_interface.kicad_sch)
- note added: "ESP32-C3-02"
- note added: "Flash Memory"
- note added: "SD Card Module"
- note added: "Test Points"
- note added: "USB module"
- title: ESP32 Sensor Board -> ESP32 - USB Module - Flash Memory - SD Card
- moved on the sheet: J3, U3, U4, U5

Commit message: clean Warnings on the SCH
Parts:
- C10, C11, C12, C13, C14, C8: footprint (none) -> Capacitor_SMD:C_0805_2012Metric_Pad1.18x1.45mm_HandSolder
- C7, C9: footprint (none) -> Capacitor_Tantalum_SMD:CP_EIA-3216-10_Kemet-I_HandSolder
- J3: footprint GSD090012SEU:AMPHENOL_GSD090012SEU -> ESP32 Project Libraries:AMPHENOL_GSD090012SEU
- LED5, LED6: footprint LEDC2012X120N -> ESP32 Project Libraries:LEDC2012X120N
- R11, R12, R13, R14, R16, R18, R19, R20, R21, R22: footprint (none) -> Resistor_SMD:R_0805_2012Metric_Pad1.20x1.40mm_HandSolder
- TP1, TP2, TP3, TP4, TP5, TP6, TP7: footprint (none) -> TestPoint:TestPoint_Pad_1.0x1.0mm
- U3: footprint ESP32-C3-WROOM-02-H4:MODULE_ESP32-C3-WROOM-02-H4 -> ESP32 Project Libraries:MODULE_ESP32-C3-WROOM-02-H4
- U4: footprint Package_DFN_QFN:SiliconLabs_QFN-20-1EP_3x3mm_P0.5mm -> Package_DFN_QFN:SiliconLabs_QFN-20-1EP_3x3mm_P0.5mm_EP1.8x1.8mm
- U6: footprint W25Q32JVSSIQ:SOIC127P790X216-8N -> ESP32 Project Libraries:SOIC127P790X216-8N

Commit message: PCB completed
Connections:
- net CS_SD: now also U3.4 (IO5); no longer U3.18 (IO0)
- net MIC_OUT: now also U3.18 (IO0); no longer U3.4 (IO5)
Changed lines of the file:
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@@
 	)
 	(label "CS_SD"
-		(at 196.85 53.34 180)
+		(at 196.85 66.04 180)
 		(effects
 			(font
@@
 	)
 	(label "MIC_OUT"
-		(at 196.85 66.04 180)
+		(at 196.85 53.34 180)
 		(effects
 			(font

Commit message: route completed
Parts:
- added H1, H2, H3, H4: MountingHole, MountingHole:MountingHole_2.5mm, symbol Mechanical:MountingHole
