File: sensors.kicad_sch (KiCad schematic)
At the start: 19 parts, among them Q1 TEMT6000X01, U2 BME280, U7 MAX4466EXK

Commit message: clean Warnings on the SCH
Parts:
- C15, C16, C18, C20, C27, C28: footprint (none) -> Capacitor_SMD:C_0805_2012Metric_Pad1.18x1.45mm_HandSolder
- MK1: footprint CMC-5042PF-AC:CUI_CMC-5042PF-AC -> ESP32 Project Libraries:CUI_CMC-5042PF-AC
- Q1: footprint TEMT6000X01:TRANS_TEMT6000X01 -> ESP32 Project Libraries:TRANS_TEMT6000X01
- R23, R24, R25, R26, R27, R28, R29, R30, R31: footprint (none) -> Resistor_SMD:R_0805_2012Metric_Pad1.20x1.40mm_HandSolder
- U2: footprint BME280:PSON65P250X250X100-8N -> ESP32 Project Libraries:PSON65P250X250X100-8N
- U7: footprint MAX4466EXK:SOT65P210X110-5N -> ESP32 Project Libraries:SOT65P210X110-5N
Changed lines of the file:
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@@
 	)
 	(junction
-		(at 203.835 80.01)
+		(at 204.47 80.01)
 		(diameter 0)
 		(color 0 0 0 0)
@@
 	)
 	(junction
-		(at 177.165 60.96)
+		(at 177.8 60.96)
 		(diameter 0)
 		(color 0 0 0 0)
@@
 	)
 	(junction
-		(at 216.535 58.42)
+		(at 217.17 58.42)
 		(diameter 0)
 		(color 0 0 0 0)
@@
 	)
 	(junction
-		(at 161.29 32.385)
+		(at 161.29 33.02)
 		(diameter 0)
 		(color 0 0 0 0)
@@
 	(wire
 		(pts
-			(xy 147.32 35.56) (xy 147.32 32.385)
+			(xy 147.32 35.56) (xy 147.32 33.02)
 		)
 		(stroke
@@
 	(wire
 		(pts
-			(xy 147.32 32.385) (xy 161.29 32.385)
+			(xy 147.32 33.02) (xy 161.29 33.02)
 		)
 		(stroke
@@
 	(wire
 		(pts
-			(xy 200.66 90.17) (xy 203.835 90.17)
+			(xy 200.66 90.17) (xy 204.47 90.17)
 		)
 		(stroke
@@
 	(wire
 		(pts
-			(xy 161.29 30.48) (xy 161.29 32.385)
+			(xy 161.29 30.48) (xy 161.29 33.02)
 		)
 		(stroke
@@
 	(wire
 		(pts
-			(xy 203.835 80.01) (xy 216.535 80.01)
+			(xy 204.47 80.01) (xy 217.17 80.01)
 		)
 		(stroke
@@
 	(wire
 		(pts
-			(xy 216.535 80.01) (xy 216.535 58.42)
+			(xy 217.17 80.01) (xy 217.17 58.42)
 		)
 		(stroke
@@
 	(wire
 		(pts
-			(xy 161.29 32.385) (xy 161.29 41.91)
+			(xy 161.29 33.02) (xy 161.29 41.91)
 		)
 		(stroke
@@
 	(wire
 		(pts
-			(xy 177.165 60.96) (xy 179.07 60.96)
+			(xy 177.8 60.96) (xy 179.07 60.96)
 		)
 		(stroke
@@
 	(wire
 		(pts
-			(xy 189.23 80.01) (xy 177.165 80.01)
+			(xy 189.23 80.01) (xy 177.8 80.01)
 		)
 		(stroke
@@
 	(wire
 		(pts
-			(xy 200.66 80.01) (xy 203.835 80.01)
+			(xy 200.66 80.01) (xy 204.47 80.01)
 		)
 		(stroke
@@
 	(wire
 		(pts
-			(xy 219.71 58.42) (xy 216.535 58.42)
+			(xy 219.71 58.42) (xy 217.17 58.42)
 		)
 		(stroke
@@
 	(wire
 		(pts
-			(xy 167.64 60.96) (xy 177.165 60.96)
+			(xy 167.64 60.96) (xy 177.8 60.96)
 		)
 		(stroke
@@
 	(wire
 		(pts
-			(xy 203.835 90.17) (xy 203.835 80.01)
+			(xy 204.47 90.17) (xy 204.47 80.01)
 		)
 		(stroke
@@
 	(wire
 		(pts
-			(xy 177.165 80.01) (xy 177.165 60.96)
+			(xy 177.8 80.01) (xy 177.8 60.96)
 		)
 		(stroke
@@
 	(wire
 		(pts
-			(xy 216.535 58.42) (xy 214.63 58.42)
+			(xy 217.17 58.42) (xy 214.63 58.42)
 		)
 		(stroke
@@
 			)
 		)
-		(property "Footprint" "BME280:PSON65P250X250X100-8N"
+		(property "Footprint" "ESP32 Project Libraries:PSON65P250X250X100-8N"
 			(at 69.85 59.69 0)
 			(effects
@@
 			)
 		)
-		(property "Footprint" ""
+		(property "Footprint" "Resistor_SMD:R_0805_2012Metric_Pad1.20x1.40mm_HandSolder"
 			(at 196.85 81.788 90)
 			(effects
@@
 			)
 		)
-		(property "Footprint" ""
+		(property "Footprint" "Resistor_SMD:R_0805_2012Metric_Pad1.20x1.40mm_HandSolder"
 			(at 159.512 45.72 90)
 			(effects
@@
 			)
 		)
-		(property "Footprint" ""
+		(property "Footprint" "Capacitor_SMD:C_0805_2012Metric_Pad1.18x1.45mm_HandSolder"
 			(at 168.6052 83.82 0)
 			(effects
@@
 			)
 		)
-		(property "Footprint" ""
+		(property "Footprint" "Resistor_SMD:R_0805_2012Metric_Pad1.20x1.40mm_HandSolder"
 			(at 29.972 53.34 90)
 			(effects
@@
 			)
 		)
-		(property "Footprint" ""
+		(property "Footprint" "Resistor_SMD:R_0805_2012Metric_Pad1.20x1.40mm_HandSolder"
 			(at 145.542 39.37 90)
 			(effects
@@
 			)
 		)
-		(property "Footprint" ""
+		(property "Footprint" "Resistor_SMD:R_0805_2012Metric_Pad1.20x1.40mm_HandSolder"
 			(at 145.542 52.07 90)
 			(effects
@@
 			)
 		)
-		(property "Footprint" "TEMT6000X01:TRANS_TEMT6000X01"
+		(property "Footprint" "ESP32 Project Libraries:TRANS_TEMT6000X01"
 			(at 81.28 121.92 0)
 			(effects
@@
 			)
 		)
-		(property "Footprint" ""
+		(property "Footprint" "Resistor_SMD:R_0805_2012Metric_Pad1.20x1.40mm_HandSolder"
 			(at 165.862 69.85 90)
 			(effects
@@
 			)
 		)
-		(property "Footprint" "CMC-5042PF-AC:CUI_CMC-5042PF-AC"
+		(property "Footprint" "ESP32 Project Libraries:CUI_CMC-5042PF-AC"
 			(at 130.81 60.96 0)
 			(effects
@@
 			)
 		)
-		(property "Footprint" ""
+		(property "Footprint" "Capacitor_SMD:C_0805_2012Metric_Pad1.18x1.45mm_HandSolder"
 			(at 193.04 91.1352 0)
 			(effects
@@
 			)
 		)
-		(property "Footprint" ""
+		(property "Footprint" "Capacitor_SMD:C_0805_2012Metric_Pad1.18x1.45mm_HandSolder"
 			(at 135.89 46.6852 0)
 			(effects
@@
 			)
 		)
-		(property "Footprint" "MAX4466EXK:SOT65P210X110-5N"
+		(property "Footprint" "ESP32 Project Libraries:SOT65P210X110-5N"
 			(at 196.85 60.96 0)
 			(effects
@@
 			)
 		)
-		(property "Footprint" ""
+		(property "Footprint" "Capacitor_SMD:C_0805_2012Metric_Pad1.18x1.45mm_HandSolder"
 			(at 151.13 59.3852 0)
 			(effects
@@
 			)
 		)
-		(property "Footprint" ""
+		(property "Footprint" "Resistor_SMD:R_0805_2012Metric_Pad1.20x1.40mm_HandSolder"
 			(at 38.862 53.34 90)
 			(effects
@@
 			)
 		)
-		(property "Footprint" ""
+		(property "Footprint" "Resistor_SMD:R_0805_2012Metric_Pad1.20x1.40mm_HandSolder"
 			(at 90.932 116.84 90)
 			(effects
@@
 			)
 		)
-		(property "Footprint" ""
+		(property "Footprint" "Resistor_SMD:R_0805_2012Metric_Pad1.20x1.40mm_HandSolder"
 			(at 159.512 69.85 90)
 			(effects
@@
 			)
 		)
-		(property "Footprint" ""
+		(property "Footprint" "Capacitor_SMD:C_0805_2012Metric_Pad1.18x1.45mm_HandSolder"
 			(at 88.5952 64.77 0)
 			(effects
@@
 			)
 		)
-		(property "Footprint" ""
+		(property "Footprint" "Capacitor_SMD:C_0805_2012Metric_Pad1.18x1.45mm_HandSolder"
 			(at 233.3752 64.77 0)
 			(effects

Commit message: PCB completed
Parts:
- added C23: 0.1u, Capacitor_SMD:C_0805_2012Metric_Pad1.18x1.45mm_HandSolder, symbol Device:C
- added C24, C25: 10n, Capacitor_SMD:C_0805_2012Metric_Pad1.18x1.45mm_HandSolder, symbol Device:C
- added R17: 35WR100KLFTR, ESP32 Project Libraries:TRIM_35WR100KLFTR, symbol 35WR100KLFTR:35WR100KLFTR
- C28: value 1u -> 10u
- R30: value 10k -> 1k
- R31: value 100k -> 22k
Connections:
- net +3.3V: now also Q1.3, C23.1; no longer R23.1
- net GND: now also R23.2, C23.2, C24.2, C25.2; no longer Q1.1
- net MIC_OUT: now also R17.1, R17.2; no longer R31.2
- net PHOTO_C: now also Q1.1, R23.1, C24.1, C25.1; no longer Q1.3, R23.2
- new net: R17.3, R31.2
Other:
- moved on the sheet: Q1, R23, R31
