File: user_interface.kicad_sch (KiCad schematic)
At the start: 11 parts, among them J4 Conn_01x04_Pin, J5 Conn_01x05_Pin, Q2 BC817, Q3 BC817

Commit message: clean Warnings on the SCH
Parts:
- C21, C22: footprint (none) -> Capacitor_SMD:C_0805_2012Metric_Pad1.18x1.45mm_HandSolder
- J4: footprint (none) -> Connector_PinHeader_2.54mm:PinHeader_1x04_P2.54mm_Vertical
- J5: footprint (none) -> Connector_PinHeader_2.54mm:PinHeader_1x05_P2.54mm_Vertical
- R33, R34, R35: footprint (none) -> Resistor_SMD:R_0805_2012Metric_Pad1.20x1.40mm_HandSolder
- S1, S2: footprint USLPT2819DT2TR:SW_USLPT2819DT2TR -> ESP32 Project Libraries:SW_USLPT2819DT2TR
Changed lines of the file:
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@@
 	)
 	(junction
-		(at 189.865 49.53)
+		(at 190.5 49.53)
 		(diameter 0)
 		(color 0 0 0 0)
 	)
 	(junction
-		(at 157.48 42.545)
+		(at 157.48 43.18)
 		(diameter 0)
 		(color 0 0 0 0)
@@
 	)
 	(junction
-		(at 151.765 110.49)
+		(at 152.4 110.49)
 		(diameter 0)
 		(color 0 0 0 0)
@@
 	)
 	(junction
-		(at 154.305 88.9)
+		(at 154.94 88.9)
 		(diameter 0)
 		(color 0 0 0 0)
@@
 	(wire
 		(pts
-			(xy 189.865 40.64) (xy 208.28 40.64)
+			(xy 190.5 40.64) (xy 208.28 40.64)
 		)
 		(stroke
@@
 	(wire
 		(pts
-			(xy 151.765 98.425) (xy 151.765 110.49)
+			(xy 152.4 99.06) (xy 152.4 110.49)
 		)
 		(stroke
@@
 	(wire
 		(pts
-			(xy 148.59 88.9) (xy 154.305 88.9)
+			(xy 148.59 88.9) (xy 154.94 88.9)
 		)
 		(stroke
@@
 	(wire
 		(pts
-			(xy 176.53 93.98) (xy 176.53 98.425)
+			(xy 176.53 93.98) (xy 176.53 99.06)
 		)
 		(stroke
@@
 	(wire
 		(pts
-			(xy 191.77 44.45) (xy 189.865 44.45)
+			(xy 191.77 44.45) (xy 190.5 44.45)
 		)
 		(stroke
@@
 	(wire
 		(pts
-			(xy 154.305 88.9) (xy 156.21 88.9)
+			(xy 154.94 88.9) (xy 156.21 88.9)
 		)
 		(stroke
@@
 	(wire
 		(pts
-			(xy 161.29 42.545) (xy 157.48 42.545)
+			(xy 161.29 43.18) (xy 157.48 43.18)
 		)
 		(stroke
@@
 	(wire
 		(pts
-			(xy 176.53 98.425) (xy 151.765 98.425)
+			(xy 176.53 99.06) (xy 152.4 99.06)
 		)
 		(stroke
@@
 	(wire
 		(pts
-			(xy 151.765 110.49) (xy 156.21 110.49)
+			(xy 152.4 110.49) (xy 156.21 110.49)
 		)
 		(stroke
@@
 	(wire
 		(pts
-			(xy 189.865 53.34) (xy 189.865 49.53)
+			(xy 190.5 53.34) (xy 190.5 49.53)
 		)
 		(stroke
@@
 	(wire
 		(pts
-			(xy 185.42 49.53) (xy 189.865 49.53)
+			(xy 185.42 49.53) (xy 190.5 49.53)
 		)
 		(stroke
@@
 	(wire
 		(pts
-			(xy 176.53 100.33) (xy 154.305 100.33)
+			(xy 176.53 100.33) (xy 154.94 100.33)
 		)
 		(stroke
@@
 	(wire
 		(pts
-			(xy 189.865 49.53) (xy 191.77 49.53)
+			(xy 190.5 49.53) (xy 191.77 49.53)
 		)
 		(stroke
@@
 	(wire
 		(pts
-			(xy 157.48 40.64) (xy 157.48 42.545)
+			(xy 157.48 40.64) (xy 157.48 43.18)
 		)
 		(stroke
@@
 	(wire
 		(pts
-			(xy 161.29 44.45) (xy 161.29 42.545)
+			(xy 161.29 44.45) (xy 161.29 43.18)
 		)
 		(stroke
@@
 	(wire
 		(pts
-			(xy 189.865 44.45) (xy 189.865 40.64)
+			(xy 190.5 44.45) (xy 190.5 40.64)
 		)
 		(stroke
@@
 	(wire
 		(pts
-			(xy 208.28 53.34) (xy 189.865 53.34)
+			(xy 208.28 53.34) (xy 190.5 53.34)
 		)
 		(stroke
@@
 	(wire
 		(pts
-			(xy 154.305 100.33) (xy 154.305 88.9)
+			(xy 154.94 100.33) (xy 154.94 88.9)
 		)
 		(stroke
@@
 	(wire
 		(pts
-			(xy 148.59 110.49) (xy 151.765 110.49)
+			(xy 148.59 110.49) (xy 152.4 110.49)
 		)
 		(stroke
@@
 	(wire
 		(pts
-			(xy 157.48 42.545) (xy 157.48 44.45)
+			(xy 157.48 43.18) (xy 157.48 44.45)
 		)
 		(stroke
@@
 			)
 		)
-		(property "Footprint" ""
+		(property "Footprint" "Resistor_SMD:R_0805_2012Metric_Pad1.20x1.40mm_HandSolder"
 			(at 160.02 112.268 90)
 			(effects
@@
 			)
 		)
-		(property "Footprint" ""
+		(property "Footprint" "Connector_PinHeader_2.54mm:PinHeader_1x05_P2.54mm_Vertical"
 			(at 81.28 95.25 0)
 			(effects
@@
 			)
 		)
-		(property "Footprint" ""
+		(property "Footprint" "Resistor_SMD:R_0805_2012Metric_Pad1.20x1.40mm_HandSolder"
 			(at 160.02 90.678 90)
 			(effects
@@
 			)
 		)
-		(property "Footprint" ""
+		(property "Footprint" "Connector_PinHeader_2.54mm:PinHeader_1x04_P2.54mm_Vertical"
 			(at 81.28 53.34 0)
 			(effects
@@
 			)
 		)
-		(property "Footprint" ""
+		(property "Footprint" "Capacitor_SMD:C_0805_2012Metric_Pad1.18x1.45mm_HandSolder"
 			(at 186.3852 59.69 0)
 			(effects
@@
 			)
 		)
-		(property "Footprint" "USLPT2819DT2TR:SW_USLPT2819DT2TR"
+		(property "Footprint" "ESP32 Project Libraries:SW_USLPT2819DT2TR"
 			(at 148.59 46.99 0)
 			(effects
@@
 			)
 		)
-		(property "Footprint" "USLPT2819DT2TR:SW_USLPT2819DT2TR"
+		(property "Footprint" "ESP32 Project Libraries:SW_USLPT2819DT2TR"
 			(at 199.39 46.99 0)
 			(effects
@@
 			)
 		)
-		(property "Footprint" ""
+		(property "Footprint" "Resistor_SMD:R_0805_2012Metric_Pad1.20x1.40mm_HandSolder"
 			(at 183.642 41.91 90)
 			(effects
@@
 			)
 		)
-		(property "Footprint" ""
+		(property "Footprint" "Capacitor_SMD:C_0805_2012Metric_Pad1.18x1.45mm_HandSolder"
 			(at 138.1252 62.23 0)
 			(effects

Commit message: SCH completed
Connections:
- net +3.3V: now also J4.4 (Pin_4); no longer J4.1 (Pin_1)
- net GND: now also J4.3 (Pin_3); no longer J4.4 (Pin_4)
- net SCL: now also J4.2 (Pin_2); no longer J4.3 (Pin_3)
- net SDA: now also J4.1 (Pin_1); no longer J4.2 (Pin_2)
Changed lines of the file:
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@@
 	(wire
 		(pts
-			(xy 140.97 44.45) (xy 139.7 44.45)
+			(xy 69.85 55.88) (xy 76.2 55.88)
 		)
 		(stroke
@@
 	(wire
 		(pts
-			(xy 71.12 97.79) (xy 76.2 97.79)
+			(xy 140.97 44.45) (xy 139.7 44.45)
 		)
 		(stroke
@@
 	(wire
 		(pts
-			(xy 69.85 55.88) (xy 76.2 55.88)
+			(xy 71.12 97.79) (xy 76.2 97.79)
 		)
 		(stroke
@@
 	(wire
 		(pts
-			(xy 163.83 88.9) (xy 168.91 88.9)
+			(xy 69.85 53.34) (xy 76.2 53.34)
 		)
 		(stroke
@@
 	(wire
 		(pts
-			(xy 137.16 49.53) (xy 140.97 49.53)
+			(xy 163.83 88.9) (xy 168.91 88.9)
 		)
 		(stroke
@@
 	(wire
 		(pts
-			(xy 71.12 100.33) (xy 71.12 104.14)
+			(xy 137.16 49.53) (xy 140.97 49.53)
 		)
 		(stroke
@@
 	(wire
 		(pts
-			(xy 176.53 93.98) (xy 176.53 99.06)
+			(xy 71.12 100.33) (xy 71.12 104.14)
 		)
 		(stroke
@@
 	(wire
 		(pts
-			(xy 191.77 44.45) (xy 190.5 44.45)
+			(xy 176.53 93.98) (xy 176.53 99.06)
 		)
 		(stroke
@@
 	(wire
 		(pts
-			(xy 69.85 58.42) (xy 69.85 62.23)
+			(xy 191.77 44.45) (xy 190.5 44.45)
 		)
 		(stroke
@@
 	(wire
 		(pts
-			(xy 69.85 44.45) (xy 69.85 50.8)
-		)
-		(stroke
-			(width 0)
-			(type default)
-		)
-	)
-	(wire
-		(pts
 			(xy 71.12 92.71) (xy 76.2 92.71)
 		)
@@
 	(wire
 		(pts
-			(xy 69.85 53.34) (xy 76.2 53.34)
-		)
-		(stroke
-			(width 0)
-			(type default)
-		)
-	)
-	(wire
-		(pts
 			(xy 185.42 49.53) (xy 190.5 49.53)
 		)
@@
 	(hierarchical_label "SDA"
 		(shape bidirectional)
-		(at 69.85 53.34 180)
+		(at 69.85 50.8 180)
 		(effects
 			(font
@@
 	(hierarchical_label "SCL"
 		(shape bidirectional)
-		(at 69.85 55.88 180)
+		(at 69.85 53.34 180)
 		(effects
 			(font
@@
 	(symbol
 		(lib_id "power:GND")
-		(at 69.85 62.23 0)
+		(at 69.85 55.88 270)
 		(unit 1)
 		(exclude_from_sim no)
@@
 		(fields_autoplaced yes)
 		(property "Reference" "#PWR042"
-			(at 69.85 68.58 0)
+			(at 63.5 55.88 0)
 			(effects
 				(font
@@
 		)
 		(property "Value" "GND"
-			(at 69.85 67.31 0)
+			(at 66.04 55.8799 90)
 			(effects
 				(font
 					(size 1.27 1.27)
 				)
+				(justify right)
 			)
 		)
 		(property "Footprint" ""
-			(at 69.85 62.23 0)
+			(at 69.85 55.88 0)
 			(effects
 				(font
@@
 		)
 		(property "Datasheet" ""
-			(at 69.85 62.23 0)
+			(at 69.85 55.88 0)
 			(effects
 				(font
@@
 		)
 		(property "Description" "Power symbol creates a global label with name \"GND\" , ground"
-			(at 69.85 62.23 0)
+			(at 69.85 55.88 0)
 			(effects
 				(font
@@
 	(symbol
 		(lib_id "power:+3.3V")
-		(at 69.85 44.45 0)
+		(at 69.85 58.42 90)
 		(unit 1)
 		(exclude_from_sim no)
@@
 		(fields_autoplaced yes)
 		(property "Reference" "#PWR056"
-			(at 69.85 48.26 0)
+			(at 73.66 58.42 0)
 			(effects
 				(font
@@
 		)
 		(property "Value" "+3.3V"
-			(at 69.85 39.37 0)
+			(at 66.04 58.4199 90)
 			(effects
 				(font
 					(size 1.27 1.27)
 				)
+				(justify left)
 			)
 		)
 		(property "Footprint" ""
-			(at 69.85 44.45 0)
+			(at 69.85 58.42 0)
 			(effects
 				(font
@@
 		)
 		(property "Datasheet" ""
-			(at 69.85 44.45 0)
+			(at 69.85 58.42 0)
 			(effects
 				(font
@@
 		)
 		(property "Description" "Power symbol creates a global label with name \"+3.3V\""
-			(at 69.85 44.45 0)
+			(at 69.85 58.42 0)
 			(effects
 				(font

Commit message: PCB completed
Parts:
- removed J5: Conn_01x05_Pin, Connector_PinHeader_2.54mm:PinHeader_1x05_P2.54mm_Vertical, symbol Connector:Conn_01x05_Pin
- added LED7: LTST-C170KRKT, ESP32 Project Libraries:LEDC2012X120N, symbol LTST-C170KRKT:LTST-C170KRKT
- added LED8: LTST-C170GKT, ESP32 Project Libraries:LEDC2012X120N, symbol LTST-C170GKT:LTST-C170GKT
- added R36: 10k, Resistor_SMD:R_0805_2012Metric_Pad1.20x1.40mm_HandSolder, symbol Device:R
- added R37, R38: 470, Resistor_SMD:R_0805_2012Metric_Pad1.20x1.40mm_HandSolder, symbol Device:R
- added S3: SW1, ESP32 Project Libraries:SW_TL3305AF260QG, symbol TL3305AF260QG:TL3305AF260QG
- S1, S2: footprint ESP32 Project Libraries:SW_USLPT2819DT2TR -> ESP32 Project Libraries:SW_TL3305AF260QG; symbol USLPT2819DT2TR:USLPT2819DT2TR -> TL3305AF260QG:TL3305AF260QG; Check_prices https://www.snapeda.com/parts/USLPT2819DT2TR/TE+Connectivit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 -> https://www.snapeda.com/parts/TL3305AF260QG/E-Switch/view-p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; MANUFACTURER TE CONNECTIVITY -> E-Switch; MAXIMUM_PACKAGE_HEIGHT (none) -> 3.8mm; MF TE Connectivity -> E-Switch; MP USLPT2819DT2TR -> TL3305AF260QG; PARTREV P -> C; Package None -> SMD-4 E-Switch; STANDARD Manufacturer Recommendations -> Manufacturer recommendations; SnapEDA_Link https://www.snapeda.com/parts/USLPT2819DT2TR/TE+Connectivit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 -> https://www.snapeda.com/parts/TL3305AF260QG/E-Switch/view-p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
Connections:
- net +3.3V: now also S3.3, S3.4
- net BOOT: now also Q3.3 (C), S1.2; no longer Q3.2 (E), S1.3
- net DTR: now also Q3.2 (E); no longer Q3.3 (C)
- net EN: now also S2.2; no longer S2.3
- net GND: now also S1.3, S2.3, R36.1, R37.2, R38.2; no longer S1.2, S2.2
- net GPIO08: now also R36.2, S3.1, S3.2
- net GPIO18: now also LED8.2 (A)
- net GPIO19: now also LED7.2 (A)
- new net: LED8.1 (K), R37.1
- new net: LED7.1 (K), R38.1
Other:
- moved on the sheet: Q2, Q3, R33, R34
